Commit message: Turning back when switching error corrected

File: src/model20/urdf/model20.urdf.xacro (robot description, xacro)
@@ -4,6 +4,6 @@
      For more information, please see http://wiki.ros.org/sw_urdf_exporter -->
 <robot
-  name="model15" xmlns:xacro="http://ros.org/wiki/xacro">
-  <xacro:arg name="laser_visual"  default="false"/>
+  name="model20" xmlns:xacro="http://ros.org/wiki/xacro">
+  <xacro:arg name="laser_visual"  default="true"/>
   <xacro:arg name="camera_visual" default="false"/>
   <xacro:arg name="imu_visual"    default="false"/>
@@ -24,8 +24,8 @@
       <inertia
         ixx="0.00338395410459643"
-        ixy="-5.22346850738525E-12"
+        ixy="-5.22346855323587E-12"
         ixz="-3.11212901639624E-05"
         iyy="0.00557048223435682"
-        iyz="1.30947753493714E-11"
+        iyz="1.30947753511968E-11"
         izz="0.00865832882623317" />
     </inertial>
@@ -36,5 +36,5 @@
       <geometry>
         <mesh
-          filename="package://model15/meshes/base_link.STL" />
+          filename="package://model20/meshes/base_link.STL" />
       </geometry>
       <material
@@ -50,5 +50,5 @@
       <geometry>
         <mesh
-          filename="package://model15/meshes/base_link.STL" />
+          filename="package://model20/meshes/base_link.STL" />
       </geometry>
     </collision>
@@ -58,12 +58,12 @@
     <inertial>
       <origin
-        xyz="0.00153023333982288 -0.00499966029225218 -6.66133814775094E-15"
-        rpy="0 0 0" />
-      <mass
-        value="0.0239463719407108" />
+        xyz="0.00153023333982283 -0.00499966029225218 -6.7168492989822E-15"
+        rpy="0 0 0" />
+      <mass
+        value="0.0239463719407107" />
       <inertia
         ixx="1.07207044697232E-06"
-        ixy="-6.56161020907689E-21"
-        ixz="1.99685049324664E-21"
+        ixy="-6.55499276417647E-21"
+        ixz="1.99761000782495E-21"
         iyy="5.97423909283024E-06"
         iyz="-3.86666262269128E-23"
@@ -76,5 +76,5 @@
       <geometry>
         <mesh
-          filename="package://model15/meshes/left_front_wheel_suspension.STL" />
+          filename="package://model20/meshes/left_front_wheel_suspension.STL" />
       </geometry>
       <material
@@ -90,5 +90,5 @@
       <geometry>
         <mesh
-          filename="package://model15/meshes/left_front_wheel_suspension.STL" />
+          filename="package://model20/meshes/left_front_wheel_suspension.STL" />
       </geometry>
     </collision>
@@ -122,6 +122,6 @@
       <inertia
         ixx="1.15503164126153E-05"
-        ixy="-2.96411876568126E-09"
-        ixz="-1.64845302072257E-08"
+        ixy="-2.96411876568134E-09"
+        ixz="-1.64845302072256E-08"
         iyy="6.93803138202261E-06"
         iyz="1.56454773172921E-07"
@@ -134,5 +134,5 @@
       <geometry>
         <mesh
-          filename="package://model15/meshes/left_front_wheel_motor.STL" />
+          filename="package://model20/meshes/left_front_wheel_motor.STL" />
       </geometry>
       <material
@@ -148,5 +148,5 @@
       <geometry>
         <mesh
-          filename="package://model15/meshes/left_front_wheel_motor.STL" />
+          filename="package://model20/meshes/left_front_wheel_motor.STL" />
       </geometry>
     </collision>
@@ -172,5 +172,5 @@
     <inertial>
       <origin
-        xyz="0.0158391990185352 -6.93889390390723E-18 3.1641356201817E-15"
+        xyz="0.0158391990185352 0 3.1641356201817E-15"
         rpy="0 0 0" />
       <mass
@@ -178,8 +178,8 @@
       <inertia
         ixx="0.0007892115763339"
-        ixy="-1.65302974455766E-20"
-        ixz="3.95755131124754E-18"
+        ixy="-1.61861562991134E-20"
+        ixz="3.95792866895153E-18"
         iyy="0.000410429434291421"
-        iyz="-3.84527315454464E-19"
+        iyz="-3.84870078420791E-19"
         izz="0.00041042943429142" />
     </inertial>
@@ -190,5 +190,5 @@
       <geometry>
         <mesh
-          filename="package://model15/meshes/left_front_wheel.STL" />
+          filename="package://model20/meshes/left_front_wheel.STL" />
       </geometry>
       <material
@@ -204,5 +204,5 @@
       <geometry>
         <mesh
-          filename="package://model15/meshes/left_front_wheel.STL" />
+          filename="package://model20/meshes/left_front_wheel.STL" />
       </geometry>
     </collision>
@@ -234,5 +234,5 @@
       <inertia
         ixx="1.07207044697232E-06"
-        ixy="-5.89903853842192E-21"
+        ixy="-5.89738417719681E-21"
         ixz="1.70976521885377E-21"
         iyy="5.97423909283023E-06"
@@ -246,5 +246,5 @@
       <geometry>
         <mesh
-          filename="package://model15/meshes/right_front_wheel_suspension.STL" />
+          filename="package://model20/meshes/right_front_wheel_suspension.STL" />
       </geometry>
       <material
@@ -260,5 +260,5 @@
       <geometry>
         <mesh
-          filename="package://model15/meshes/right_front_wheel_suspension.STL" />
+          filename="package://model20/meshes/right_front_wheel_suspension.STL" />
       </geometry>
     </collision>
@@ -286,5 +286,5 @@
     <inertial>
       <origin
-        xyz="-2.79575138501104E-05 0.0019490794439902 -0.012936461929631"
+        xyz="-2.79575138501173E-05 0.00194907944399023 -0.012936461929631"
         rpy="0 0 0" />
       <mass
@@ -292,17 +292,17 @@
       <inertia
         ixx="1.15503164126153E-05"
-        ixy="-2.9641187656836E-09"
-        ixz="-1.64845302071878E-08"
+        ixy="-2.96411876568394E-09"
+        ixz="-1.64845302071881E-08"
         iyy="6.93803138202261E-06"
         iyz="1.56454773172925E-07"
-        izz="9.57898906372989E-06" />
-    </inertial>
-    <visual>
-      <origin
-        xyz="0 0 0"
-        rpy="0 0 0" />
-      <geometry>
-        <mesh
-          filename="package://model15/meshes/right_front_wheel_motor.STL" />
+        izz="9.5789890637299E-06" />
+    </inertial>
+    <visual>
+      <origin
+        xyz="0 0 0"
+        rpy="0 0 0" />
+      <geometry>
+        <mesh
+          filename="package://model20/meshes/right_front_wheel_motor.STL" />
       </geometry>
       <material
@@ -318,5 +318,5 @@
       <geometry>
         <mesh
-          filename="package://model15/meshes/right_front_wheel_motor.STL" />
+          filename="package://model20/meshes/right_front_wheel_motor.STL" />
       </geometry>
     </collision>
@@ -342,5 +342,5 @@
     <inertial>
       <origin
-        xyz="0.0158391990185491 1.31838984174237E-16 1.94289029309402E-16"
+        xyz="0.0158391990185491 1.2490009027033E-16 1.94289029309402E-16"
         rpy="0 0 0" />
       <mass
@@ -348,6 +348,6 @@
       <inertia
         ixx="0.0007892115763339"
-        ixy="-1.3297776936908E-20"
-        ixz="-1.31191060294497E-18"
+        ixy="-1.3086845880707E-20"
+        ixz="-1.31197073179041E-18"
         iyy="0.000410429434291421"
         iyz="-3.30739896123204E-19"
@@ -360,5 +360,5 @@
       <geometry>
         <mesh
-          filename="package://model15/meshes/right_front_wheel.STL" />
+          filename="package://model20/meshes/right_front_wheel.STL" />
       </geometry>
       <material
@@ -374,5 +374,5 @@
       <geometry>
         <mesh
-          filename="package://model15/meshes/right_front_wheel.STL" />
+          filename="package://model20/meshes/right_front_wheel.STL" />
       </geometry>
     </collision>
@@ -404,8 +404,8 @@
       <inertia
         ixx="4.29479133591148E-06"
-        ixy="8.8579111407478E-10"
-        ixz="1.01813691673353E-09"
+        ixy="8.85791114074875E-10"
+        ixz="1.01813691673291E-09"
         iyy="2.21058141232447E-05"
-        iyz="2.1757968121536E-08"
+        iyz="2.17579681215362E-08"
         izz="2.35707058046399E-05" />
     </inertial>
@@ -416,5 +416,5 @@
       <geometry>
         <mesh
-          filename="package://model15/meshes/camera.STL" />
+          filename="package://model20/meshes/camera.STL" />
       </geometry>
       <material
@@ -430,5 +430,5 @@
       <geometry>
         <mesh
-          filename="package://model15/meshes/camera.STL" />
+          filename="package://model20/meshes/camera.STL" />
       </geometry>
     </collision>
@@ -451,5 +451,5 @@
     <inertial>
       <origin
-        xyz="-5.92450278861234E-05 -0.0201677348757047 0.000391328969376853"
+        xyz="-5.92450278861234E-05 -0.0201677348757047 0.000391328969376881"
         rpy="0 0 0" />
       <mass
@@ -457,8 +457,8 @@
       <inertia
         ixx="0.000426495369649312"
-        ixy="-1.33941181513932E-07"
-        ixz="-1.32777557424162E-06"
+        ixy="-1.33941181513931E-07"
+        ixz="-1.32777557424163E-06"
         iyy="0.000584026336355448"
-        iyz="-9.7817502168308E-08"
+        iyz="-9.78175021683085E-08"
         izz="0.000183119671370759" />
     </inertial>
@@ -469,5 +469,5 @@
       <geometry>
         <mesh
-          filename="package://model15/meshes/myrio.STL" />
+          filename="package://model20/meshes/myrio.STL" />
       </geometry>
       <material
@@ -483,5 +483,5 @@
       <geometry>
         <mesh
-          filename="package://model15/meshes/myrio.STL" />
+          filename="package://model20/meshes/myrio.STL" />
       </geometry>
     </collision>
@@ -504,23 +504,23 @@
     <inertial>
       <origin
-        xyz="-5.69397911324709E-05 0.0158670533538898 0.055083544841935"
-        rpy="0 0 0" />
-      <mass
-        value="0.399542896482383" />
-      <inertia
-        ixx="0.000432029127757847"
-        ixy="-1.833831243821E-07"
-        ixz="-3.17164967884077E-07"
-        iyy="0.000836965270422519"
-        iyz="4.77447001747385E-07"
-        izz="0.000473016843887474" />
-    </inertial>
-    <visual>
-      <origin
-        xyz="0 0 0"
-        rpy="0 0 0" />
-      <geometry>
-        <mesh
-          filename="package://model15/meshes/intel.STL" />
+        xyz="-5.69397911358849E-05 0.0158670533538911 0.0550835448419378"
+        rpy="0 0 0" />
+      <mass
+        value="0.399542896482345" />
+      <inertia
+        ixx="0.000432029127757804"
+        ixy="-1.83383124401157E-07"
+        ixz="-3.17164967926806E-07"
+        iyy="0.000836965270422433"
+        iyz="4.7744700176345E-07"
+        izz="0.000473016843887417" />
+    </inertial>
+    <visual>
+      <origin
+        xyz="0 0 0"
+        rpy="0 0 0" />
+      <geometry>
+        <mesh
+          filename="package://model20/meshes/intel.STL" />
       </geometry>
       <material
@@ -536,5 +536,5 @@
       <geometry>
         <mesh
-          filename="package://model15/meshes/intel.STL" />
+          filename="package://model20/meshes/intel.STL" />
       </geometry>
     </collision>
@@ -544,6 +544,6 @@
     type="fixed">
     <origin
-      xyz="0.20552 -0.10937 -0.025995"
-      rpy="1.5708 -0.0058285 0" />
+      xyz="0.205522597365492 -0.109366659682657 -0.0259953857991605"
+      rpy="1.5707963267949 -0.00582847831492263 0" />
     <parent
       link="base_link" />
@@ -563,6 +563,6 @@
       <inertia
         ixx="0.000357684284600866"
-        ixy="-3.61913558197252E-09"
-        ixz="-2.92942384657856E-07"
+        ixy="-3.61913558197348E-09"
+        ixz="-2.92942384657851E-07"
         iyy="0.000746477971691014"
         iyz="4.03533275235886E-06"
@@ -575,5 +575,5 @@
       <geometry>
         <mesh
-          filename="package://model15/meshes/nvidia.STL" />
+          filename="package://model20/meshes/nvidia.STL" />
       </geometry>
       <material
@@ -589,5 +589,5 @@
       <geometry>
         <mesh
-          filename="package://model15/meshes/nvidia.STL" />
+          filename="package://model20/meshes/nvidia.STL" />
       </geometry>
     </collision>
@@ -597,6 +597,6 @@
     type="fixed">
     <origin
-      xyz="0.41837 -0.19195 0.036381"
-      rpy="-1.5766 0 -1.5708" />
+      xyz="0.418367655264176 -0.191953362348841 0.0363810058695082"
+      rpy="-1.57662480510981 0 -1.5707963267949" />
     <parent
       link="base_link" />
@@ -610,23 +610,23 @@
     <inertial>
       <origin
-        xyz="1.6791266697791E-05 -0.0504338842827013 -0.00500218320308373"
-        rpy="0 0 0" />
-      <mass
-        value="0.295010921800958" />
-      <inertia
-        ixx="0.000699646991202319"
-        ixy="1.57075731798077E-08"
-        ixz="-1.74299199713213E-09"
-        iyy="0.00218325621057825"
-        iyz="-1.62706054100039E-09"
-        izz="0.00275998123079568" />
-    </inertial>
-    <visual>
-      <origin
-        xyz="0 0 0"
-        rpy="0 0 0" />
-      <geometry>
-        <mesh
-          filename="package://model15/meshes/pusher .STL" />
+        xyz="4.88473400367395E-07 -0.0465265708699117 0.0229929210393978"
+        rpy="0 0 0" />
+      <mass
+        value="0.22688114098655" />
+      <inertia
+        ixx="0.000430709062315012"
+        ixy="-1.19594594798727E-09"
+        ixz="-5.02913337951274E-12"
+        iyy="0.000930442337810295"
+        iyz="-3.21405921052249E-05"
+        izz="0.00127031110351361" />
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
Commit message: Added IMU, modified README

File: src/model20/urdf/model20.urdf.xacro (robot description, xacro)
@@ -1446,3 +1446,38 @@
     </sensor>
   </gazebo>
+  <gazebo reference="imu">
+    <sensor type="imu" name="imu">
+      <always_on>true</always_on>
+      <visualize>$(arg imu_visual)</visualize>
+    </sensor>
+    <material>Gazebo/Grey</material>
+  </gazebo>
+  <gazebo>
+    <plugin name="imu_plugin" filename="libgazebo_ros_imu.so">
+      <alwaysOn>true</alwaysOn>
+      <bodyName>imu</bodyName>
+      <frameName>imu</frameName>
+      <topicName>imu</topicName>
+      <serviceName>imu_service</serviceName>
+      <gaussianNoise>0.0</gaussianNoise>
+      <updateRate>200</updateRate>
+      <imu>
+        <noise>
+          <type>gaussian</type>
+          <rate>
+            <mean>0.0</mean>
+            <stddev>2e-4</stddev>
+            <bias_mean>0.0000075</bias_mean>
+            <bias_stddev>0.0000008</bias_stddev>
+          </rate>
+          <accel>
+            <mean>0.0</mean>
+            <stddev>1.7e-2</stddev>
+            <bias_mean>0.1</bias_mean>
+            <bias_stddev>0.001</bias_stddev>
+          </accel>
+        </noise>
+      </imu>
+    </plugin>
+  </gazebo>
 </robot>
